File: AntennaPCB.kicad_pcb (KiCad board)
At the start: 2 copper layers, 500.3 x 102.3 mm, 32 parts, among them J1 Conn_Coaxial, J10 Conn_01x06_Pin, J11 Conn_01x06_Pin, J12 Conn_01x06_Pin, J13 Conn_01x06_Pin, J14 Conn_01x06_Pin, J15 Conn_01x06_Pin, J16 Conn_01x06_Pin, J2 Conn_Coaxial, J3 Conn_Coaxial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

Commit message: Fixed the antenna
Parts:
- U1, U2, U3, U4, U5, U6, U7, U8: footprint userLibPersonal:Antenna Element -> Userlib:Antenna element
- moved U1 12.8 mm to (55.6, 45.0)
- moved U2 12.8 mm to (118.1, 45.0)
- moved U3 12.8 mm to (180.6, 45.0)
- moved U4 12.8 mm to (243.1, 45.0)
- moved U5 12.8 mm to (305.6, 45.0)
- moved U6 12.8 mm to (368.1, 45.0)
- moved U7 12.8 mm to (430.6, 45.0)
- moved U8 12.8 mm to (493.1, 45.0)
