File: AntennaPCB.kicad_sch (KiCad schematic)
At the start: 32 parts, among them J1 Conn_Coaxial, J10 Conn_01x06_Pin, J11 Conn_01x06_Pin, J12 Conn_01x06_Pin, J13 Conn_01x06_Pin, J14 Conn_01x06_Pin, J15 Conn_01x06_Pin, J16 Conn_01x06_Pin, J2 Conn_Coaxial, J3 Conn_Coaxial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

Commit message: Fixed the antenna
Parts:
- U1, U2, U3, U4, U5, U6, U7, U8: footprint userLibPersonal:Antenna Element -> Userlib:Antenna element
Changed lines of the file:
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@@
       (effects (font (size 1.27 1.27)))
     )
-    (property "Footprint" "userLibPersonal:Antenna Element" (at 83.82 44.45 0)
+    (property "Footprint" "Userlib:Antenna element" (at 83.82 44.45 0)
       (effects (font (size 1.27 1.27)) hide)
     )
@@
       (effects (font (size 1.27 1.27)))
     )
-    (property "Footprint" "userLibPersonal:Antenna Element" (at 45.72 44.45 0)
+    (property "Footprint" "Userlib:Antenna element" (at 45.72 44.45 0)
       (effects (font (size 1.27 1.27)) hide)
     )
@@
       (effects (font (size 1.27 1.27)))
     )
-    (property "Footprint" "userLibPersonal:Antenna Element" (at 60.96 44.45 0)
+    (property "Footprint" "Userlib:Antenna element" (at 60.96 44.45 0)
       (effects (font (size 1.27 1.27)) hide)
     )
@@
       (effects (font (size 1.27 1.27)))
     )
-    (property "Footprint" "userLibPersonal:Antenna Element" (at 76.2 44.45 0)
+    (property "Footprint" "Userlib:Antenna element" (at 76.2 44.45 0)
       (effects (font (size 1.27 1.27)) hide)
     )
@@
       (effects (font (size 1.27 1.27)))
     )
-    (property "Footprint" "userLibPersonal:Antenna Element" (at 38.1 44.45 0)
+    (property "Footprint" "Userlib:Antenna element" (at 38.1 44.45 0)
       (effects (font (size 1.27 1.27)) hide)
     )
@@
       (effects (font (size 1.27 1.27)))
     )
-    (property "Footprint" "userLibPersonal:Antenna Element" (at 68.58 44.45 0)
+    (property "Footprint" "Userlib:Antenna element" (at 68.58 44.45 0)
       (effects (font (size 1.27 1.27)) hide)
     )
@@
       (effects (font (size 1.27 1.27)))
     )
-    (property "Footprint" "userLibPersonal:Antenna Element" (at 53.34 44.45 0)
+    (property "Footprint" "Userlib:Antenna element" (at 53.34 44.45 0)
       (effects (font (size 1.27 1.27)) hide)
     )
@@
       (effects (font (size 1.27 1.27)))
     )
-    (property "Footprint" "userLibPersonal:Antenna Element" (at 91.44 44.45 0)
-      (effects (font (size 1.27 1.27)) hide)
-    )
+    (property "Footprint" "Userlib:Antenna element" (at 91.44 44.45 0)
+      (effects (font (size 1.27 1.27)) hide)
+    )
